File: pcb/rail.crossing.brd (EAGLE design)
At the start: 60.8 x 24 mm, 26 parts, among them IC1 LM386M-1, Q1 BC847SMD, U1 ATTINY85V-10SU, U2 LM1117MP-5.0

Commit message: add new board witch mask
Parts:
- removed C6: 100uF, rcl:SMC_C
- removed JP3: (no value), jumper:JP7SMD
- added C5: (no value), rcl:SMC_D
- added JP4: (no value), pinhead:2X04/90
- added JP5: (no value), pinhead:2X03/90
- added JP6: (no value), pinhead:1X03/90
- added JP7: (no value), pinhead:1X02/90
- added SJ2: (no value), jumper:SJ
- JP2: device jumper:JP6SMD -> pinhead:1X02/90
- moved JP2 12.0 mm to (79.7, 60.5)
- moved R4 1.68 mm to (67.2, 45.4), turned to 90 degrees
- moved LED1 1.21 mm to (64.6, 45.5)
- moved U1 0.56 mm to (64.8, 55.9)
- moved R5 0.56 mm to (63.9, 60.0)
- moved C1 0.34 mm to (64.4, 63.1)
- moved U2 0.27 mm to (36.3, 59.2)
Connections:
- removed net N$23: C4.1, JP2.P$3, LED1.A, R2.2, R4.2, U1.8, U2.2
- new net N$15: JP5.3, JP5.4, LED1.A, R2.2, R4.2, SJ2.2, U1.8
- new net N$20: C4.1, SJ2.1, U2.2
- net JP1: now also JP6.1; no longer JP3.P$1
- net JP2: now also JP5.1, JP5.2, JP6.3; no longer C6.-, JP2.P$2, JP3.P$3
- net N$10: now also JP5.5, JP5.6; no longer JP2.P$4
- net N$11: now also JP7.2; no longer JP2.P$6
- net N$12: now also JP4.1, JP4.2; no longer JP3.P$4
- net N$14: now also JP7.1; no longer JP2.P$5
- net N$21: now also JP6.2; no longer JP3.P$2
- net N$22: now also C5.+; no longer C6.+
- net RED1: now also JP2.2, JP4.5, JP4.6; no longer JP3.P$6
- net RED2: now also JP4.3, JP4.4; no longer JP3.P$5
- net WHITE: now also JP2.1, JP4.7, JP4.8; no longer JP2.P$1, JP3.P$7
Routing:
- net N$23: track 80.5 -> 0.00 mm, vias 1 -> 0
- net N$15: track 0.00 -> 74.6 mm, vias 0 -> 1
- net RED1: track 51.8 -> 73.6 mm
- net N$20: track 0.00 -> 6.13 mm
- net JP2: track 150.9 -> 155.8 mm
- net WHITE: track 68.1 -> 71.5 mm
- net S$1: track 3.30 -> 0.00 mm
- net N$11: track 37.6 -> 35.2 mm, vias 2 -> 0
- net JP1: track 42.7 -> 44.3 mm
- net N$21: track 8.97 -> 10.2 mm
- net N$10: track 8.86 -> 10.00 mm
- net N$12: track 11.0 -> 12.1 mm
- net N$14: track 43.2 -> 44.2 mm
- net N$22: track 23.2 -> 22.3 mm
- net N$17: track 17.9 -> 18.6 mm, vias 2 -> 4
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Other:
- board size 60.8 x 24 mm -> 72.9 x 46.2 mm
- board text added: "+ R1 R2 WH"
- board text added: "+12V"
- board text added: "+5V LED"
- board text added: "+5V SERVO"
- board text added: "-12V"
- board text added: "-5V SERVO"
- board text added: "BÍLÁ"
- board text added: "BÍLÁ LED"
- board text added: "GND"
- board text added: "IZOLOVANÁ KOLEJ"
- board text added: "KOLEJIŠTĚ, -12V"
- board text added: "MOSI"
- board text added: "REPRO"
- board text added: "RST"
- board text added: "SERVO"
- board text added: "SERVO SIGNÁL"
- board text added: "ČERNÁ"
- board text added: "ČERVENÁ"
- board text added: "ČERVENÁ LED1"
- board text added: "ČERVENÁ LED2"
