File: pcb/rail.crossing.sch (EAGLE design)
At the start: 26 parts, among them IC1 LM386M-1, Q1 BC847SMD, U1 ATTINY85V-10SU, U2 LM1117MP-5.0

Commit message: add new board witch mask
Parts:
- removed C6: 100uF, rcl:CPOL-EUSMCC
- removed JP3: J7SMD, jumper:J7SMD
- added C5: (no value), rcl:CPOL-EUSMCD
- added JP4: (no value), pinhead:PINHD-2X4/90
- added JP5: (no value), pinhead:PINHD-2X3/90
- added JP6: (no value), pinhead:PINHD-1X3/90
- added JP7: (no value), pinhead:PINHD-1X2/90
- added SJ2: (no value), jumper:SJ
- JP2: value J6SMD -> (none); device jumper:J6SMD -> pinhead:PINHD-1X2/90
Connections:
- removed net N$23: C4.1, JP2.3, LED1.A, R2.2, R4.2, U1.VCC, U2.OUT
- new net N$15: JP5.3, JP5.4, LED1.A, R2.2, R4.2, SJ2.2, U1.VCC
- new net N$20: C4.1, SJ2.1, U2.OUT
- net JP1: now also JP6.1; no longer JP3.1
- net JP2: now also JP5.1, JP5.2, JP6.3; no longer C6.-, JP2.2, JP3.3
- net N$10: now also JP5.5, JP5.6; no longer JP2.4
- net N$11: now also JP7.2; no longer JP2.6
- net N$12: now also JP4.1, JP4.2; no longer JP3.4
- net N$14: now also JP7.1; no longer JP2.5
- net N$21: now also JP6.2; no longer JP3.2
- net N$22: now also C5.+; no longer C6.+
- net RED1: now also JP2.2, JP4.5, JP4.6; no longer JP3.6
- net RED2: now also JP4.3, JP4.4; no longer JP3.5
- net WHITE: now also JP4.7, JP4.8; no longer JP3.7
